File: schematics/v1.2/SRAM Board 2MB.kicad_pcb (KiCad board)
At the start: 2 copper layers, 125.7 x 30.5 mm, 47 parts, among them J1 Conn_01x01, J10 Conn_01x01, J11 Conn_01x01, J12 Conn_01x01, J13 Conn_01x01, J14 Conn_01x01, J15 Conn_01x01, J16 Conn_01x01, J17 Conn_01x01, J18 Conn_01x01, J19 Conn_01x01, J2 Conn_01x01, J20 Conn_01x01, J21 Conn_01x01, J22 Conn_01x01, J23 Conn_01x01, J24 Conn_01x01, J25 Conn_01x01, J26 Conn_01x01, J27 Conn_01x01, J28 Conn_01x01, J29 Conn_01x01, J3 Conn_01x01, J30 Conn_01x01, J31 Conn_01x01, J32 Conn_01x01, J4 Conn_01x01, J5 Conn_01x01, J6 Conn_01x01, J7 Conn_01x01, J8 Conn_01x01, J9 Conn_01x01, U1 74ABT821ADW, U2 74ABT00, U3 AS7C316098B-10TIN, U34 74LS373, U4 74ABT373, U7 LM1117-3.3

Commit message: Add files via upload
Parts:
- removed C9: 10uF, Capacitor_SMD:C_1206_3216Metric_Pad1.42x1.75mm_HandSolder
- removed the U2 at (176.5, 90.2)
- removed U7: LM1117-3.3, Package_TO_SOT_SMD:SOT-223
- added U1: 74ABT00, Package_SO:SOIC-14_3.9x8.7mm_P1.27mm, F.Cu at (174.6, 93.9)
- added U4: CY62157ESL-45ZSXI, Package_SO:TSOP-II-44_10.16x18.41mm_P0.8mm_copy, F.Cu at (190.6, 91.9)
- added U5: CY62157ESL-45ZSXI, Package_SO:TSOP-II-44_10.16x18.41mm_P0.8mm_copy, F.Cu at (212.7, 91.9)
- C8: value 10uF -> 0.1uF
- U3: value AS7C316098B-10TIN -> 74ABT32; footprint Package_SO:TSOP-II-54_22.2x10.16mm_P0.8mm -> Package_SO:SOIC-14_3.9x8.7mm_P1.27mm
- moved C3 48.9 mm to (156.7, 78.0)
- moved C4 41.0 mm to (162.4, 78.0)
- moved C8 27.6 mm to (198.9, 77.9)
- moved C5 20.0 mm to (193.2, 74.0)
- moved C7 20.0 mm to (193.2, 77.9)
- moved C6 17.5 mm to (198.9, 74.0)
- moved U3 10.9 mm to (184.2, 77.5)
- moved U2 1.51 mm to (162.4, 90.7)
- moved C1 0.18 mm to (156.7, 74.2)
- moved C2 0.18 mm to (162.4, 74.2)
- renumbered U1 to U2, U4 to U6
Connections:
- C3 pad 1: /vcc33 -> /vcc5
- C4 pad 1: /vcc33 -> /vcc5
- C5 pad 1: /vcc33 -> /vcc5
- C6 pad 1: /vcc33 -> /vcc5
- C7 pad 1: /vcc33 -> /vcc5
- U3 pad 1: /d12 -> /_sramce
- U3 pad 10: /ma1 -> (no net)
- U3 pad 11: /ma0 -> (no net)
- U3 pad 12: /_ucas -> (no net)
- U3 pad 13: /_sramce -> (no net)
- U3 pad 14: /vcc33 -> /vcc5
- U3 pad 2: /vcc33 -> /_invbdra9
- U3 pad 3: /d13 -> /_ceu4
- U3 pad 4: /d14 -> /_sramce
- U3 pad 5: /gnd -> /bdra9
- U3 pad 6: /d15 -> /_ceu5
- U3 pad 7: /ma4 -> /gnd
- U3 pad 8: /ma3 -> (no net)
- U3 pad 9: /ma2 -> (no net)
- U34 pad 2: /1q -> /bdra9
- U34 pad 3: /dra9 -> /1d
- U6 pad 2: /1q -> /bdra9
- U6 pad 3: /dra9 -> /1d
Routing:
- net /vcc5: track 0.00 -> 305.6 mm
- net /gnd: track 0.00 -> 280.2 mm, vias 0 -> 5
- net /bdra9: track 0.00 -> 169.2 mm, vias 0 -> 2
- net /a2: track 0.00 -> 138.0 mm, vias 0 -> 1
- net /a8: track 0.00 -> 129.1 mm, vias 0 -> 4
- net /a1: track 0.00 -> 117.2 mm, vias 0 -> 1
- net /a5: track 0.00 -> 111.6 mm
- net /a0: track 0.00 -> 108.6 mm, vias 0 -> 1
- net /d13: track 0.00 -> 105.8 mm, vias 0 -> 2
- net /d15: track 0.00 -> 103.4 mm, vias 0 -> 2
- net /a3: track 0.00 -> 101.9 mm, vias 0 -> 2
- net /a7: track 0.00 -> 101.3 mm, vias 0 -> 2
- net /a4: track 0.00 -> 97.3 mm, vias 0 -> 1
- net /a6: track 0.00 -> 96.4 mm, vias 0 -> 1
- net /_we: track 0.00 -> 91.5 mm, vias 0 -> 1
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Other:
- board size 125.7 x 30.5 mm -> 125.7 x 33 mm
- board text added: "/bras0"
- board text added: "/bras1"
- board text added: "/lcas"
- board text added: "/ucas"
- board text added: "/we"
- board text added: "1"
- board text added: "74ABT32"
- board text added: "8Mb (512K x 16) SRAM"
- board text added: "CY62157ESL-45ZSXI"
- board text added: "Quad 2-input OR Gate"
- board text added: "a0"
- board text added: "a1"
- board text added: "a2"
- board text added: "a3"
- board text added: "a4"
- board text added: "a5"
- board text added: "a6"
- board text added: "a7"
- board text added: "a8"
- board text added: "d0"
- board text added: "d1"
- board text added: "d10"
- board text added: "d11"
- board text added: "d12"
- board text added: "d13"
- board text added: "d14"
- board text added: "d15"
- board text added: "d2"
- board text added: "d3"
- board text added: "d4"
- board text added: "d5"
- board text added: "d6"
- board text added: "d7"
- board text added: "d8"
- board text added: "d9"
- board text added: "gnd"
- board text added: "vcc"
- board text removed: "16Mb (1024K x 16) SRAM"
- board text removed: "3.3v Decoupling Capacitors"
- board text removed: "3.3v Linear Regulator"
